File: examples/output/schematic/Arduino_最小系统板__ATmega328P_PU_.kicad_sch (KiCad schematic)
At the start: 8 parts, among them U1 ATmega328P-P, Y1 16MHz

Commit message: fix: 真实LLM模式自纠错 + 原理图渲染/布局/文字重叠修复 (ERC 0错误0警告)
真实LLM模式:
- netlist_generator: 网表提示词锁定位号(禁止臆造); 自纠错回落(引用BOM不存在的位号/符号不存在的引脚时丢弃对应连接而非崩溃); 错误回灌
- bom_generator: _check_symbols 校验symbol存在性, suggest_lib_id 自动纠正假符号(Device:SW_Push->Switch:SW_Push, LM1117-5.0->LM1117T-5.0)后直接返回
- symbol_lib: 新增 pin_names/list_symbols/suggest_lib_id; 内嵌符号定义扁平化(消除extends导致原理图加载失败); 嵌套单元符号名不带库前缀
- validator: 缺失位号提示补充BOM实际位号, 回灌更精准

原理图渲染(kicad_writer):
- 修复Y轴翻转(库Y向上->原理图Y向下), 引出线方向正确
- 逐列紧凑布局(按高度降序装箱, A4装不下升A3), 消除元件画到页外/挤成一坨
- 引脚引出线25.4->7.62mm, 杜绝不同网络导线共线重叠(VCC/GND曾被误合并)
- PWR_FLAG碰撞检测放置 + 文字隐藏; 同网邻近端点互连只挂一个标签, 消除VCC×VCC文字叠压
- 未连接引脚打no_connect, 单引脚网络不再悬空标签
- knowledge: mock网表R2:2重复入网修正; mock分支补validate_netlist

验证: mock与真实数据两份原理图 ERC 均 0错误 0警告, 文字重叠0对
Parts:
- removed C1, C2: 22pF, symbol C
- removed C3: 100nF, symbol C
- removed D1: LED, symbol LED
- removed R1: 10k, symbol R
- removed R2: 330, symbol R
- removed U1: ATmega328P-P, Package_DIP:DIP-28_W11.18mm, symbol ATmega328P-P
- removed Y1: 16MHz, symbol Crystal
- added C1, C2: 22pF, symbol Device:C
- added C3: 100nF, symbol Device:C
- added D1: LED, symbol Device:LED
- added R1: 10k, symbol Device:R
- added R2: 330, symbol Device:R
- added U1: ATmega328P-P, symbol MCU_Microchip_ATmega:ATmega328P-P
- added Y1: 16MHz, symbol Device:Crystal
Connections:
- net GND: now also C1.2, C2.2, C3.2, D1.2 (A), U1.22 (GND), U1.8 (GND)
- new net LED: D1.1 (K), R2.2
- new net RESET: R1.2, U1.1 (~{RESET}/PC6)
- new net VCC: C3.1, R1.1, R2.1, U1.20 (AVCC), U1.7 (VCC)
- new net XTAL1: C1.1, U1.9 (XTAL1/PB6), Y1.1
- new net XTAL2: C2.1, U1.10 (XTAL2/PB7), Y1.2
- no-connect marks 0 -> 21
